File: DAC7578Breakout/DAC7578Breakout.kicad_pcb (KiCad board)
At the start: 2 copper layers, 26.4 x 22.9 mm, 11 parts, among them J1 Conn_01x08, J2 Conn_01x08, U1 DAC7578

Commit message: Readme and silkscreen
Other:
- board text added: "A"
- board text added: "ADDR0"
- board text added: "B"
- board text added: "C"
- board text added: "D"
- board text added: "E"
- board text added: "F"
- board text added: "G"
- board text added: "GND"
- board text added: "H"
- board text added: "NCLR"
- board text added: "NLDAC"
- board text added: "SCL"
- board text added: "SDA"
- board text added: "VIN"
