File: DAC7578Breakout/DAC7578Breakout.kicad_sch (KiCad schematic)
At the start: 11 parts, among them J1 Conn_01x08, J2 Conn_01x08, U1 DAC7578

Commit message: Readme and silkscreen
Other:
- note added: "Connectors"
- note removed: "Vout Connector"
- note removed: "mbed Connector"
- moved on the sheet: C1, J1, J2, R1, R2
